Commit message: find solution for a given Q

File: descriptions/robot_descriptions/objects_description/objects/bottle.urdf (robot description, URDF)
Before this commit: robot bottle, 2 links, 1 joints
Links:
- link bottle: geometry collision cylinder length=18 radius=3; visual mesh filename=package://objects_description/meshes/visual/bottle.obj scale=1.0 1.0 1.0

Commit message: sync

File: descriptions/robot_descriptions/objects_description/objects/bottle.urdf (robot description, URDF)
Before this commit: robot bottle, 2 links, 1 joints
Links:
- link bottle: geometry visual mesh filename=package://objects_description/meshes/visual/bottle.obj scale=1.0 1.0 1.0
Joints:
- joint bottle_to_world: origin xyz=0 0 0 rpy=0 0 0 -> xyz=0 0 0 rpy=0 1.57 0

File: descriptions/robot_descriptions/objects_description/objects/water_bottle.urdf (robot description, URDF)
Before this commit: robot bottle, 2 links, 1 joints
Links:
- removed link bottle
- removed link world
- added link baseLink
- added link bottle_head, mass 0.032; collision mesh filename=package://objects_description/meshes/visual/water_bottle_bo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 scale=1.0 1.0 1.0; visual mesh filename=package://objects_description/meshes/visual/water_bottle_bo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 scale=1.0 1.0 1.0
- added link bottle_water, mass 0.173; collision mesh filename=package://objects_description/meshes/visual/water_bottle_wa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 scale=1.0 1.0 1.0; visual mesh filename=package://objects_description/meshes/visual/water_bottle_wa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 scale=1.0 1.0 1.0
Joints:
- added joint bottle_filled_water: type fixed, parent bottle_head, child bottle_water, origin xyz=0 0 0 rpy=0 0 0
- joint bottle_to_world: child bottle -> bottle_head; origin xyz=0 0 0 rpy=0 0 0 -> xyz=0 0 0 rpy=-1.57 0 0; parent world -> baseLink
