Commit message: modify the bottle description

File: descriptions/robot_descriptions/objects_description/objects/water_bottle.urdf (robot description, URDF)
Before this commit: robot filled_bottle, 3 links, 2 joints
Links:
- removed link bottle_head
- removed link bottle_water
- added link body, mass 0.042; collision mesh filename=package://objects_description/meshes/visual/water_bottle_bo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 scale=1.0 1.0 1.0; visual mesh filename=package://objects_description/meshes/visual/water_bottle_bo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 scale=1.0 1.0 1.0
- added link cap, mass 0.012; collision mesh filename=package://objects_description/meshes/visual/water_bottle_ca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 scale=1.0 1.0 1.0; visual mesh filename=package://objects_description/meshes/visual/water_bottle_ca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 scale=1.0 1.0 1.0
- added link water, mass 0.1536; collision mesh filename=package://objects_description/meshes/visual/water_bottle_wa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 scale=1.0 1.0 1.0; visual mesh filename=package://objects_description/meshes/visual/water_bottle_wa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 scale=1.0 1.0 1.0
Joints:
- removed joint bottle_filled_water
- removed joint bottle_to_world
- added joint bottle_body: type fixed, parent cap, child body, origin xyz=0 0 0 rpy=0 0 0
- added joint bottle_cap: type fixed, parent baseLink, child cap, origin xyz=0 0 -225 rpy=1.57 0 0
- added joint bottle_water: type fixed, parent cap, child water, origin xyz=0 0 0 rpy=0 0 0
